File: OBQAS/OBQAS.kicad_sch (KiCad schematic)
At the start: 146 parts, among them J1 24V IN, J2 USB_C_Receptacle_USB2.0, J3 K type, J5 TF_PUSH, J6 CH1, J7 CH2, K1 G5NB-1A-E_DC5, K2 G5NB-1A-E_DC5, K3 G5NB-1A-E_DC5, K4 G5NB-1A-E_DC5, Q1 IRLML2803TRPBF, Q2 IRLML2803TRPBF, Q3 IRLML2803TRPBF, Q4 IRLML2803TRPBF, Q5 BC846, Q6 BC846, Q7 IRLZ44N, Q8 IRLZ44N, Q9 IRFP064, SW1 SW_SPST, SW2 Enc, U1 LM7805_TO220, U2 AMS1117-3.3, U3 ESP32-WROOM-32, U4 CH340C, U5 TPS55288QWRPMRQ1, U6 LM358, U7 LM358, U8 MCP4921, U9 ADS1115IDGS

Commit message: additional schematic changes to accommodate balancing
Parts:
- added BZ?: Buzzer, symbol Device:Buzzer
- added J?: Conn_01x03, symbol Connector_Generic:Conn_01x03
- added J?: Conn_01x06, symbol Connector_Generic:Conn_01x06
- added J?: Conn_01x05, symbol Connector_Generic:Conn_01x05
- added J?: Conn_01x04, symbol Connector_Generic:Conn_01x04
- added Q?: IRLML2803TRPBF, Package_TO_SOT_SMD:SOT-23, symbol IRLML2803TRPBF:IRLML2803TRPBF
- added Q?: BC846, Package_TO_SOT_SMD:SOT-23, symbol Transistor_BJT:BC846
- added R? (x2): 470, Resistor_SMD:R_0805_2012Metric_Pad1.20x1.40mm_HandSolder, symbol Device:R
- added R? (x5): 1k, Resistor_SMD:R_0805_2012Metric_Pad1.20x1.40mm_HandSolder, symbol Device:R
- added R?: 100, Resistor_SMD:R_0805_2012Metric_Pad1.20x1.40mm_HandSolder, symbol Device:R
- added R? (x4): 10k, Resistor_SMD:R_0805_2012Metric_Pad1.20x1.40mm_HandSolder, symbol Device:R
- added R?: 5.1k, Resistor_SMD:R_0805_2012Metric_Pad1.20x1.40mm_HandSolder, symbol Device:R
- added U?: PCF8574, symbol Interface_Expansion:PCF8574
Connections:
- net +3V3: now also R?.1, R?.2, R?.2, R?.2, R?.2, R?.2, U?.16 (VDD)
- net ADC_READY: now also U?.10 (P5); no longer U3.26 (IO4)
- net CH1R1_SIG: now also R?.1, U?.7 (P3); no longer U3.9 (IO33)
- net CH1R2_SIG: now also R?.1, U?.6 (P2); no longer U3.8 (IO32)
- net CH2R1_SIG: now also R?.1, U?.5 (P1); no longer U3.12 (IO27)
- net CH2R2_SIG: now also R?.1, U?.4 (P0); no longer U3.11 (IO26)
- net DAC_LDAC: now also U?.12 (P7); no longer U3.27 (IO16)
- net ENC_Button: now also U?.11 (P6); no longer U3.14 (IO12)
- net EN_UVLDO: now also R?.1, U?.9 (P4); no longer U3.24 (IO2)
- net GND: now also J?.1 (Pin_1), J?.1 (Pin_1), J?.1 (Pin_1), J?.1 (Pin_1), Q?.2, Q?.2 (E), R?.1, R?.2, U?.1 (A0), U?.2 (A1), U?.3 (A2), U?.8 (VSS)
- net SCL: now also U?.15 (SDA)
- net SDA: now also U?.14 (SCL)
- new net: Q?.1, R?.1, R?.1
- new net: J?.2 (Pin_2), J?.2 (Pin_2), J?.2 (Pin_2), J?.2 (Pin_2), R?.2, R?.2
- new net: J?.3 (Pin_3), J?.3 (Pin_3), J?.3 (Pin_3), J?.3 (Pin_3)
- new net: J?.4 (Pin_4), J?.4 (Pin_4), J?.4 (Pin_4)
- new net: J?.5 (Pin_5), J?.5 (Pin_5)
- new net: Q?.1 (B), R?.2, R?.2
- new net: Q?.3, R?.1
- new net: Q?.3 (C), R?.1
- new net 1S_ADC: R?.1, R?.2
- new net PCF_INT: R?.2, U3.24 (IO2), U?.13 (~{INT})
- no-connect marks 16 -> 14
Other:
- note added: "fix op amp common mode"
- note added: "set these to balance transistors and use esp for relay ones"
- note added: "use large resistors?"
