File: OBQAS/OBQAS.kicad_sch (KiCad schematic)
At the start: 167 parts, among them J1 24V IN, J2 USB_C_Receptacle_USB2.0, J3 K type, J5 TF_PUSH, J6 CH1, J7 CH2, K1 G5NB-1A-E_DC5, K2 G5NB-1A-E_DC5, K3 G5NB-1A-E_DC5, K4 G5NB-1A-E_DC5, Q1 IRLML2803TRPBF, Q2 IRLML2803TRPBF, Q3 IRLML2803TRPBF, Q4 IRLML2803TRPBF, Q5 BC846, Q6 BC846, Q7 IRLZ44N, Q8 IRLZ44N, Q9 IRFP064, SW1 SW_SPST, SW2 Enc, U1 LM7805_TO220, U2 AMS1117-3.3, U3 ESP32-WROOM-32, U4 CH340C, U5 TPS55288QWRPMRQ1, U6 LM358, U7 LM358, U8 MCP4921, U9 ADS1115IDGS

Commit message: updated schematic with balancing circuit
Parts:
- removed Q?: IRLML2803TRPBF, Package_TO_SOT_SMD:SOT-23, symbol IRLML2803TRPBF:IRLML2803TRPBF
- removed Q?: BC846, Package_TO_SOT_SMD:SOT-23, symbol Transistor_BJT:BC846
- removed R5, R? (x2): 470, Resistor_SMD:R_0805_2012Metric_Pad1.20x1.40mm_HandSolder, symbol Device:R
- removed R? (x5): 1k, Resistor_SMD:R_0805_2012Metric_Pad1.20x1.40mm_HandSolder, symbol Device:R
- removed R?: 100, Resistor_SMD:R_0805_2012Metric_Pad1.20x1.40mm_HandSolder, symbol Device:R
- removed R? (x3): 10k, Resistor_SMD:R_0805_2012Metric_Pad1.20x1.40mm_HandSolder, symbol Device:R
- removed R?: 5.1k, Resistor_SMD:R_0805_2012Metric_Pad1.20x1.40mm_HandSolder, symbol Device:R
- added C23, C24, C26: 10u, Capacitor_SMD:C_1206_3216Metric_Pad1.33x1.80mm_HandSolder, symbol Device:C
- added C25, C27, C28, C29, C30, C31: 100n, Capacitor_SMD:C_0805_2012Metric_Pad1.18x1.45mm_HandSolder, symbol Device:C
- added C32: 1000u, Capacitor_THT:CP_Radial_D10.0mm_P5.00mm, symbol Device:C_Polarized
- added D6: 1N4001, Diode_SMD:D_SOD-123, symbol Diode:1N4001
- added L2: 22uH, Inductor_SMD:L_6.3x6.3_H3, symbol Device:L
- added Q10, Q11, Q12, Q13, Q14: IRLML2803TRPBF, Package_TO_SOT_SMD:SOT-23, symbol IRLML2803TRPBF:IRLML2803TRPBF
- added R63: 1k, Resistor_SMD:R_0805_2012Metric_Pad1.20x1.40mm_HandSolder, symbol Device:R
- added R64, R65: 5.1k, Resistor_SMD:R_0805_2012Metric_Pad1.20x1.40mm_HandSolder, symbol Device:R
- added R66, R67, R69, R71, R73, R74, R75, R87, R89: 10k, Resistor_SMD:R_0805_2012Metric_Pad1.20x1.40mm_HandSolder, symbol Device:R
- added R68, R70, R86, R88, R9: 50k, Resistor_SMD:R_0805_2012Metric_Pad1.20x1.40mm_HandSolder, symbol Device:R
- added R72: 20k, Resistor_SMD:R_0805_2012Metric_Pad1.20x1.40mm_HandSolder, symbol Device:R
- added R76, R77, R78, R81: 100, Resistor_SMD:R_0805_2012Metric_Pad1.20x1.40mm_HandSolder, symbol Device:R
- added R79, R80, R83, R84, R85: 10, Resistor_SMD:R_2512_6332Metric_Pad1.40x3.35mm_HandSolder, symbol Device:R
- added R82: 100, Inductor_SMD:L_0805_2012Metric_Pad1.15x1.40mm_HandSolder, symbol Device:R
- added U11: MT3608, Package_TO_SOT_SMD:SOT-23-6, symbol Regulator_Switching:MT3608
- added U12: LM7824_TO220, Package_TO_SOT_THT:TO-220-3_Vertical, symbol Regulator_Linear:LM7824_TO220
- added U13, U14, U15, U16, U17: HY2213-BB3A, HY2213:SOT95P280X140-6N, symbol HY2213-BB3A:HY2213-BB3A
- BZ1: renamed from BZ?; footprint (none) -> Buzzer_Beeper:Buzzer_12x9.5RM7.6
- J1: value 24V IN -> 24V MAX
- J10: renamed from J?; footprint (none) -> Connector_JST:JST_XH_B6B-XH-A_1x06_P2.50mm_Vertical
- J4: renamed from J?; footprint (none) -> Connector_JST:JST_XH_B3B-XH-A_1x03_P2.50mm_Vertical
- J8: renamed from J?; footprint (none) -> Connector_JST:JST_XH_B4B-XH-A_1x04_P2.50mm_Vertical
- J9: renamed from J?; footprint (none) -> Connector_JST:JST_XH_B5B-XH-A_1x05_P2.50mm_Vertical
- U10: renamed from U?; footprint (none) -> Package_SO:SOIC-16W_7.5x10.3mm_P1.27mm
- gave numbers to parts that had none: 1
Connections:
- net +3V3: now also U6.5 (+)
- net +5V: now also R6.2; no longer U7.8 (V+)
- net 1S_ADC: now also U3.26 (IO4), R74.1, R75.2
- net CH1R1_SIG: now also U3.9 (IO33); no longer U10.7 (P3)
- net CH1R2_SIG: now also U3.8 (IO32); no longer U10.6 (P2)
- net CH1_ADC_I: now also R88.2; no longer U9.6 (AIN2)
- net CH2R1_SIG: now also U3.12 (IO27); no longer U10.5 (P1)
- net CH2R2_SIG: now also U3.11 (IO26); no longer U10.4 (P0)
- net CH2_ADC_I: now also R86.2; no longer U9.7 (AIN3)
- net GND: now also J10.6 (Pin_6), J4.3 (Pin_3), J8.4 (Pin_4), J9.5 (Pin_5), C23.1, C24.2, C25.2, C26.2, C30.2, C32.2, Q13.2, R63.1, R65.2, R67.1, R69.1, R71.1, R73.1, R75.1, R87.2, R89.2, U11.2 (GND), U12.2 (GND), U16.3 (VSS); no longer J10.1 (Pin_1), J4.1 (Pin_1), J8.1 (Pin_1), J9.1 (Pin_1), R6.2
- net TPS_OUT: now also C32.1
- net VCC: now also C23.2, L2.1, U11.4 (EN), U11.5 (IN)
- net at BZ1.1 (-): now also R6.1
- net at BZ1.2 (+): now also U10.4 (P0)
- net BAT_1S: now reaches J10.5 (Pin_5)
- net BAT_1S: now also J4.2 (Pin_2), J8.3 (Pin_3), J9.4 (Pin_4), C31.2, Q14.2, R81.2, R84.2, U17.3 (VSS); no longer J9.5 (Pin_5)
- net 2S_ADC: now reaches U3.14 (IO12)
- net 2S_ADC: now also R72.1, R73.2
- net 3S_ADC: now reaches U3.27 (IO16)
- net 3S_ADC: now also R70.1, R71.2
- net 4S_ADC: now reaches U3.6 (IO34)
- net 4S_ADC: now also R68.1, R69.2
- net 5S_ADC: now reaches U3.7 (IO35)
- net 5S_ADC: now also R66.1, R67.2
- net +2V5 renamed +12V
- net +12V: now also R64.2, R65.1; no longer R6.1, U6.5 (+)
- new net: Q12.3, R83.1
- new net: R63.2, R9.1, U11.3 (FB)
- new net: C27.1, R76.1, U13.2 (VDD)
- new net: R88.1, R89.1, U9.6 (AIN2)
- new net: R86.1, R87.1, U9.7 (AIN3)
- new net: C24.1, C25.1, D6.1 (K), R9.2, U12.1 (VI)
- new net: C28.1, R77.1, U14.2 (VDD)
- new net: C31.1, R82.1, U17.2 (VDD)
- new net: Q14.3, R85.1
- new net: C29.1, R78.1, U15.2 (VDD)
- new net: Q10.3, R79.1
- new net: C30.1, R81.1, U16.2 (VDD)
- new net: D6.2 (A), L2.2, U11.1 (SW)
- new net: Q11.3, R80.1
- new net: Q13.3, R84.1
- new net +24V: C26.1, R64.1, U12.3 (VO), U7.8 (V+)
- new net 1S_SENSE: Q13.1, R74.2, U16.6 (OUT)
- new net 2S_SENSE: Q14.1, R72.2, U17.6 (OUT)
- new net 3S_SENSE: Q11.1, R70.2, U14.6 (OUT)
- new net 4S_SENSE: Q10.1, R68.2, U13.6 (OUT)
- new net 5S_SENSE: Q12.1, R66.2, U15.6 (OUT)
- new net BAT_2S: C28.2, J10.4 (Pin_4), J4.1 (Pin_1), J8.2 (Pin_2), J9.3 (Pin_3), Q11.2, R82.2, R85.2, U14.3 (VSS)
- new net BAT_3S: C27.2, J10.3 (Pin_3), J8.1 (Pin_1), J9.2 (Pin_2), Q10.2, R77.2, R80.2, U13.3 (VSS)
- new net BAT_4S: C29.2, J10.2 (Pin_2), J9.1 (Pin_1), Q12.2, R76.2, R79.2, U15.3 (VSS)
- new net BAT_5S: J10.1 (Pin_1), R78.2, R83.2
- no-connect marks 14 -> 32
Other:
- note added: "Vin ▲ | | | | | R1 | | |_| |---► Vout | | | | R2 | | |_| | --- GND"
- note added: "doing PWM via I2C would be inefficent, but we don't need to beep that often"
- note added: "max ADC vin -> 3.3V 1S -> Vmax 4.4V R1=10k R2=10k Vout=2.2V 2S -> Vmax 8.8V R1=20k R2=10k Vout=2.9V 3S -> Vmax 13.2V R1=50k R2=10k Vout=2.2V 4S -> Vmax 17.6V R1=50k R2=10k Vout=2.9V 5S -> Vmax 22.0V R1=50k R2=5.1k Vout=2.0V"
- note removed: "set these to balance transistors and use esp for relay ones"
- note removed: "use large resistors?"
- moved on the sheet: BZ1, C20, J5, R35, R40, R46, R52, R58, U7C
