File: OBQAS/OBQAS.kicad_pcb (KiCad board)
At the start: 2 copper layers, 151 x 118 mm, 204 parts, among them J1 24V MAX, J10 Conn_01x06, J2 USB_C_Receptacle_USB2.0, J3 K type, J4 Conn_01x03, J5 TF_PUSH, J6 CH1, J7 CH2, J8 Conn_01x04, J9 Conn_01x05, K1 G5NB-1A-E_DC5, K2 G5NB-1A-E_DC5, K3 G5NB-1A-E_DC5, K4 G5NB-1A-E_DC5, Q1 IRLML2803TRPBF, Q10 IRLML2803TRPBF, Q11 IRLML2803TRPBF, Q12 IRLML2803TRPBF, Q13 IRLML2803TRPBF, Q14 IRLML2803TRPBF, Q2 IRLML2803TRPBF, Q3 IRLML2803TRPBF, Q4 IRLML2803TRPBF, Q5 BC846, Q6 BC846, Q7 IRLZ44N, Q8 IRLZ44N, Q9 IRFP064, SW1 SW_SPST, SW2 Enc, U1 LM7805_TO220, U10 PCF8574, U11 MT3608, U12 LM7824_TO220, U13 HY2213-BB3A, U14 HY2213-BB3A, U15 HY2213-BB3A, U16 HY2213-BB3A, U17 HY2213-BB3A, U2 AMS1117-3.3, U3 ESP32-WROOM-32, U4 CH340C, U5 TPS55288QWRPMRQ1, U6 LM358, U7 LM358, U8 MCP4921, U9 ADS1115IDGS

Commit message: smal tweaks to the PCB
Other:
- board text added: "2004 I2C display"
- board text added: "Antenna Keep-out"
- board text added: "OBQAS rev 0.1 Dmytro Feb 2022"

Commit message: added gerbers
Other:
- outline, holes or cut-outs redrawn
- board text added: "JLCJLCJLCJLC"
- board text added: "OBQAS rev 0.1 DDL Feb 2022"
- board text removed: "OBQAS rev 0.1 Dmytro Feb 2022"
